Commit message: dump

File: franka_description/robots/common/franka_robot.xacro (robot description, xacro)
@@ -56,4 +56,5 @@
          tip="${arm_id}_joint8"
        />
+      <xacro:transmission-franka-pose arm_id="${arm_id}" ee_joint="${arm_id}_joint8" />
       <xacro:if value="${hand}">
         <xacro:gazebo-joint joint="${arm_id}_finger_joint1" transmission="hardware_interface/EffortJointInterface" />

File: franka_description/robots/common/utils.xacro (robot description, xacro)
@@ -198,4 +198,15 @@
     </transmission>
   </xacro:macro>
+  <xacro:macro name="transmission-franka-pose" params="arm_id:=panda ee_joint:=panda_joint8">
+    <transmission name="${arm_id}_franka_pose_cartesian">
+      <type>franka_hw/FrankaPoseCartesianInterface</type>
+      <joint name="${ee_joint}">
+        <hardwareInterface>franka_hw/FrankaPoseCartesianInterface</hardwareInterface>
+      </joint>
+      <actuator name="${ee_joint}_actuator">
+        <hardwareInterface>franka_hw/FrankaPoseCartesianInterface</hardwareInterface>
+      </actuator>
+    </transmission>
+  </xacro:macro>
   <xacro:macro name="inertia-cylinder" params="mass radius h">
     <inertial>

Commit message: depth cam integration

File: franka_description/robots/common/franka_robot.xacro (robot description, xacro)
@@ -1,5 +1,5 @@
 <?xml version='1.0' encoding='utf-8'?>
 <robot xmlns:xacro="http://www.ros.org/wiki/xacro">
-  <xacro:macro name="franka_robot" params="arm_id joint_limits parent:='world' xyz:='0 0 0' rpy:='0 0 0' hand:=false gazebo:=false tcp_xyz:='0 0 0.1034' tcp_rpy='0 0 0'">
+  <xacro:macro name="franka_robot" params="arm_id joint_limits parent:='world' xyz:='0 0 0' rpy:='0 0 0' hand:=false gazebo:=false camera:=true tcp_xyz:='0 0 0.1034' tcp_rpy='0 0 0'">
     <xacro:include filename="$(find franka_description)/robots/common/utils.xacro" />
     <xacro:include filename="$(find franka_description)/robots/common/franka_arm.xacro" />
@@ -51,8 +51,18 @@
       <xacro:gazebo-joint joint="${arm_id}_joint6" transmission="hardware_interface/EffortJointInterface" />
       <xacro:gazebo-joint joint="${arm_id}_joint7" transmission="hardware_interface/EffortJointInterface" />
+    <xacro:if value="${camera}">
+      <link name="${arm_id}_camera_link_fix"/>
+      <joint name="${arm_id}_camera_joint_fix" type="fixed">
+        <parent link="${arm_id}_link7"/>
+        <child link="${arm_id}_camera_link_fix"/>
+        <origin xyz="0.05 0.0 0.1159" rpy="0 0 ${-pi/4}"/>
+      </joint>
+      <xacro:include filename="$(find franka_description)/robots/common/depth_camera.urdf.xacro" />
+      <xacro:depth_camera arm_id="${arm_id}" connected_to="${arm_id}_camera_link_fix" />
+    </xacro:if>
       <xacro:transmission-franka-state arm_id="${arm_id}" />
       <xacro:transmission-franka-model arm_id="${arm_id}"
-         root="${arm_id}_joint1"
-         tip="${arm_id}_joint8"
+        root="${arm_id}_joint1"
+        tip="${arm_id}_joint8"
        />
       <xacro:transmission-franka-pose arm_id="${arm_id}" ee_joint="${arm_id}_joint8" />
