Commit message: suction depth incorporated

File: franka_description/robots/common/depth_camera.urdf.xacro (robot description, xacro)
@@ -1,4 +1,4 @@
 <robot xmlns:xacro="http://www.ros.org/wiki/xacro">
-  <xacro:macro name="depth_camera" params="connected_to arm_id">
+  <xacro:macro name="depth_camera" params="connected_to arm_id pos:='0 0 0' rpy:='${pi} ${-pi/2} 0'">
     <link name="${arm_id}_camera_link">
       <visual>
@@ -23,5 +23,5 @@
       <parent link="${connected_to}"/>
       <child link="${arm_id}_camera_link"/>
-      <origin xyz="0 0 0" rpy="${pi} ${-pi/2} 0"/>
+      <origin xyz="${pos}" rpy="${rpy}"/>
     </joint>
     <link name="${arm_id}_camera_depth_frame"/>

File: franka_description/robots/common/franka_pump.xacro (robot description, xacro)
@@ -1,5 +1,5 @@
 <?xml version='1.0' encoding='utf-8'?>
 <robot xmlns:xacro="http://www.ros.org/wiki/xacro" name="franka_combined">
-  <xacro:macro name="franka_robot" params="arm_id joint_limits parent:='world' xyz:='0 0 0' rpy:='0 0 0' gazebo:=false tcp_xyz:='0 0 0.1034' tcp_rpy='0 0 0'">
+  <xacro:macro name="franka_robot" params="arm_id joint_limits parent:='world' xyz:='0 0 0' rpy:='0 0 0' gazebo:=false camera:=true tcp_xyz:='0 0 0.1034' tcp_rpy='0 0 0'">
     <!-- Include Franka utils and arm -->
     <xacro:include filename="$(find franka_description)/robots/common/utils.xacro" />
@@ -94,4 +94,14 @@
       <xacro:gazebo-joint joint="${arm_id}_joint6" transmission="hardware_interface/EffortJointInterface" />
       <xacro:gazebo-joint joint="${arm_id}_joint7" transmission="hardware_interface/EffortJointInterface" />
+      <xacro:if value="${camera}">
+        <link name="${arm_id}_camera_link_fix"/>
+        <joint name="${arm_id}_camera_joint_fix" type="fixed">
+          <parent link="${arm_id}_link7"/>
+          <child link="${arm_id}_camera_link_fix"/>
+          <origin xyz="0 0 0" rpy="0 0 ${-pi/4}"/>
+        </joint>
+        <xacro:include filename="$(find franka_description)/robots/common/depth_camera.urdf.xacro" />
+        <xacro:depth_camera arm_id="${arm_id}" connected_to="${arm_id}_camera_link_fix" pos="0.055 0.0 0.15"/>
+      </xacro:if>
       <xacro:transmission-franka-state arm_id="${arm_id}" />
       <xacro:transmission-franka-model arm_id="${arm_id}"

File: franka_description/robots/common/franka_robot.xacro (robot description, xacro)
@@ -56,8 +56,8 @@
         <parent link="${arm_id}_link7"/>
         <child link="${arm_id}_camera_link_fix"/>
-        <origin xyz="0.05 0.0 0.1159" rpy="0 0 ${-pi/4}"/>
+        <origin xyz="0 0 0" rpy="0 0 ${-pi/4}"/>
       </joint>
       <xacro:include filename="$(find franka_description)/robots/common/depth_camera.urdf.xacro" />
-      <xacro:depth_camera arm_id="${arm_id}" connected_to="${arm_id}_camera_link_fix" />
+      <xacro:depth_camera arm_id="${arm_id}" connected_to="${arm_id}_camera_link_fix" pos="0.033 0.0 0.15"/>
     </xacro:if>
       <xacro:transmission-franka-state arm_id="${arm_id}" />
